File: Board/TeslaBMBCheck/TeslaBMBCheck.kicad_pcb (KiCad board)
At the start: 2 copper layers, 0 parts

Commit message: Board & schematic
Parts:
- added C1: 100n, Capacitor_SMD:C_0805_2012Metric, F.Cu at (141.7, 60.5)
- added C15: 22p, Capacitor_SMD:C_0805_2012Metric, F.Cu at (147.4, 87.9)
- added C17: 22p, Capacitor_SMD:C_0805_2012Metric, F.Cu at (138.4, 87.9)
- added C2: 10u, Capacitor_SMD:C_1206_3216Metric, F.Cu at (163.1, 71.6)
- added C3: 100n, Capacitor_SMD:C_0805_2012Metric, F.Cu at (86.4, 69.8)
- added C4: 100n, Capacitor_SMD:C_0805_2012Metric, F.Cu at (86.4, 83.9)
- added C5: 1u, Capacitor_SMD:C_0805_2012Metric, F.Cu at (128.1, 86.4)
- added C6: 47n, Capacitor_SMD:C_0805_2012Metric, F.Cu at (83.7, 101.2)
- added D15: INFO, LED_SMD:LED_0805_2012Metric, F.Cu at (114.5, 101.7)
- added DS1: WC1602A, spetry:LCD-20x4, B.Cu at (125.3, 77.7)
- added J1: TESLA_BMS, spetry:Molex_Mini-Fit_Jr_5566-10A_1x05_P4.20mm_Vertical, F.Cu at (89.4, 96.6)
- added J9: ICSP, Connector_PinHeader_2.54mm:PinHeader_1x05_P2.54mm_Vertical, F.Cu at (170.7, 79.8)
- added Q1: IRLML2244, Package_TO_SOT_SMD:SOT-23, F.Cu at (132.2, 81.8)
- added Q2: BSS138, Package_TO_SOT_SMD:SOT-23, F.Cu at (126.0, 56.0)
- added R1: 5K1, Resistor_SMD:R_0805_2012Metric, F.Cu at (161.5, 63.0)
- added R10: 22K, Resistor_SMD:R_0805_2012Metric, F.Cu at (151.9, 56.9)
- added R19: 1K, Resistor_SMD:R_0805_2012Metric, F.Cu at (124.1, 81.7)
- added R2: 5K1, Resistor_SMD:R_0805_2012Metric, F.Cu at (161.5, 67.1)
- added R23: 10K, Resistor_SMD:R_0805_2012Metric, F.Cu at (166.1, 80.8)
- added R3: 4K7, Resistor_SMD:R_0805_2012Metric, F.Cu at (121.9, 73.2)
- added R4: 4K7, Resistor_SMD:R_0805_2012Metric, F.Cu at (126.0, 73.2)
- added R5: 4K7, Resistor_SMD:R_0805_2012Metric, F.Cu at (111.4, 95.0)
- added R6: 22, Resistor_SMD:R_0805_2012Metric, F.Cu at (128.1, 81.8)
- added R8: 10K, Resistor_SMD:R_0805_2012Metric, F.Cu at (126.0, 61.5)
- added REF**: MountingHole_3mm, MountingHole:MountingHole_3mm, F.Cu at (78.2, 105.2)
- added REF**: MountingHole_3mm, MountingHole:MountingHole_3mm, F.Cu at (171.7, 50.3)
- added REF**: MountingHole_3mm, MountingHole:MountingHole_3mm, F.Cu at (78.2, 50.3)
- added REF**: MountingHole_3mm, MountingHole:MountingHole_3mm, F.Cu at (171.7, 105.2)
- added RV1: 10K, Potentiometer_SMD:Potentiometer_Bourns_TC33X_Vertical, F.Cu at (158.7, 57.3)
- added SW1: ~, Button_Switch_SMD:SW_SPST_CK_RS282G05A3, F.Cu at (80.8, 66.9)
- added SW2: ~, Button_Switch_SMD:SW_SPST_CK_RS282G05A3, F.Cu at (80.8, 83.1)
- added U1: USBLC6, Package_TO_SOT_SMD:SOT-23-6, F.Cu at (123.3, 66.7)
- added U2: PIC18F2480-ISO, Package_SO:SOIC-28W_7.5x17.9mm_P1.27mm, F.Cu at (139.1, 69.2)
- added USB1: POWER, spetry:HRO-TYPE-C-31-M-12, F.Cu at (174.4, 65.0)
- added Y1: 10 MHz, Crystal:Crystal_SMD_HC49-SD, F.Cu at (142.9, 82.3)
Routing:
- net VCC: track 0.00 -> 163.1 mm, vias 0 -> 8
- net /BMS_TX: track 0.00 -> 92.4 mm
- net /BMS_RX: track 0.00 -> 82.3 mm
- net /VPP: track 0.00 -> 72.0 mm
- net /BMS_VCC: track 0.00 -> 67.4 mm
- net Net-(U2-RA1/AN1): track 0.00 -> 61.0 mm
- net Net-(D15-K): track 0.00 -> 60.0 mm
- net Net-(U2-RA0/AN0): track 0.00 -> 54.3 mm
- net /PGD: track 0.00 -> 53.1 mm
- net /PGC: track 0.00 -> 50.5 mm
- net /LCD_RS: track 0.00 -> 47.9 mm, vias 0 -> 2
- net Net-(D15-A): track 0.00 -> 43.4 mm
- net /LCD_E: track 0.00 -> 40.8 mm
- net BACKLT: track 0.00 -> 30.5 mm
- net GND: track 0.00 -> 25.4 mm, vias 0 -> 19
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- added copper zone on B.Cu, net GND
Other:
- board outline added: 99.4 x 60.2 mm
- board text added: "CONTRAST"
- board text added: "FAULT"
- board text added: "GND"
- board text added: "ICSP"
- board text added: "POWER"
- board text added: "RX"
- board text added: "Rev 0.1 2025"
- board text added: "TX"
- board text added: "Tesla BMB Connector Pinout"
- board text added: "TeslaBMBChecker"
- board text added: "VCC"
- board text added: "github.com/svpetry/TeslaBMBCheck"

Commit message: Change info LED connection
Parts:
- moved R19 25.4 mm to (147.4, 91.7), turned to 180 degrees
Connections:
- D15 pad 1: Net-(D15-K) -> GND
- R19 pad 1: VCC -> Net-(U2-CCP1/RC2)
- U2 pad 13: Net-(D15-K) -> Net-(U2-CCP1/RC2)
Routing:
- net Net-(D15-K): track 60.0 -> 0.00 mm
- net Net-(U2-CCP1/RC2): track 0.00 -> 22.4 mm
- net Net-(D15-A): track 43.4 -> 35.8 mm
- net VCC: track 163.1 -> 159.1 mm
- net GND: track 25.4 -> 26.5 mm, vias 19 -> 20
Changed lines of the file:
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@@
 	)
 	(paper "A4")
+	(title_block
+		(title "TeslaBMBChecker")
+		(date "2025-07-10")
+		(rev "0.1")
+	)
 	(layers
 		(0 "F.Cu" signal)
@@
 	(net 42 "unconnected-(USB1-SBU1-Pad9)")
 	(net 43 "Net-(D15-A)")
-	(net 44 "Net-(D15-K)")
+	(net 44 "Net-(U2-CCP1{slash}RC2)")
 	(footprint "Package_TO_SOT_SMD:SOT-23"
 		(layer "F.Cu")
@@
 			(layers "F.Cu" "F.Mask" "F.Paste")
 			(roundrect_rratio 0.25)
-			(net 44 "Net-(D15-K)")
+			(net 1 "GND")
 			(pinfunction "K")
 			(pintype "passive")
@@
 	(footprint "Resistor_SMD:R_0805_2012Metric"
 		(layer "F.Cu")
-		(at 124.1044 81.7372 -90)
+		(at 147.447 91.694 180)
 		(descr "Resistor SMD 0805 (2012 Metric), square (rectangular) end terminal, IPC-7351 nominal, (Body size source: IPC-SM-782 page 72, https://www.pcb-3d.com/wordpress/wp-content/uploads/ipc-sm-782a_amendment_1_and_2.pdf), generated with kicad-footprint-generator")
 		(tags "resistor")
 		(property "Reference" "R19"
-			(at 0 1.6515 90)
+			(at 0 1.6515 0)
 			(layer "F.SilkS")
 			(effects
@@
 		)
 		(property "Value" "1K"
-			(at 0 1.65 90)
+			(at 0 1.65 0)
 			(layer "F.Fab")
 			(effects
@@
 		)
 		(property "Datasheet" ""
-			(at 0 0 90)
+			(at 0 0 0)
 			(layer "F.Fab")
 			(hide yes)
@@
 		)
 		(property "Description" ""
-			(at 0 0 90)
+			(at 0 0 0)
 			(layer "F.Fab")
 			(hide yes)
@@
 		)
 		(fp_line
-			(start -1.68 0.95)
-			(end -1.68 -0.95)
+			(start 1.68 0.95)
+			(end -1.68 0.95)
 			(stroke
 				(width 0.05)
@@
 		)
 		(fp_line
-			(start 1.68 0.95)
-			(end -1.68 0.95)
+			(start 1.68 -0.95)
+			(end 1.68 0.95)
 			(stroke
 				(width 0.05)
@@
 		)
 		(fp_line
-			(start -1.68 -0.95)
-			(end 1.68 -0.95)
+			(start -1.68 0.95)
+			(end -1.68 -0.95)
 			(stroke
 				(width 0.05)
@@
 		)
 		(fp_line
-			(start 1.68 -0.95)
-			(end 1.68 0.95)
+			(start -1.68 -0.95)
+			(end 1.68 -0.95)
 			(stroke
 				(width 0.05)
@@
 		)
 		(fp_line
-			(start -1 0.625)
-			(end -1 -0.625)
+			(start 1 0.625)
+			(end -1 0.625)
 			(stroke
 				(width 0.1)
@@
 		)
 		(fp_line
-			(start 1 0.625)
-			(end -1 0.625)
+			(start 1 -0.625)
+			(end 1 0.625)
 			(stroke
 				(width 0.1)
@@
 		)
 		(fp_line
-			(start -1 -0.625)
-			(end 1 -0.625)
+			(start -1 0.625)
+			(end -1 -0.625)
 			(stroke
 				(width 0.1)
@@
 		)
 		(fp_line
-			(start 1 -0.625)
-			(end 1 0.625)
+			(start -1 -0.625)
+			(end 1 -0.625)
 			(stroke
 				(width 0.1)
@@
 		)
 		(fp_text user "${REFERENCE}"
-			(at 0 0 90)
+			(at 0 0 0)
 			(layer "F.Fab")
 			(effects
@@
 		)
 		(pad "1" smd roundrect
-			(at -0.9125 0 270)
+			(at -0.9125 0 180)
 			(size 1.025 1.4)
 			(layers "F.Cu" "F.Mask" "F.Paste")
 			(roundrect_rratio 0.243902)
-			(net 2 "VCC")
+			(net 44 "Net-(U2-CCP1{slash}RC2)")
 			(pintype "passive")
 		)
 		(pad "2" smd roundrect
-			(at 0.9125 0 270)
+			(at 0.9125 0 180)
 			(size 1.025 1.4)
 			(layers "F.Cu" "F.Mask" "F.Paste")
@@
 			(layers "F.Cu" "F.Mask" "F.Paste")
 			(roundrect_rratio 0.25)
-			(net 44 "Net-(D15-K)")
+			(net 44 "Net-(U2-CCP1{slash}RC2)")
 			(pinfunction "CCP1/RC2")
 			(pintype "bidirectional")
@@
 	)
 	(segment
+		(start 114.5032 103.7082)
+		(end 114.554 103.759)
+		(width 0.25)
+		(layer "F.Cu")
+		(net 1)
+	)
+	(segment
 		(start 122.1795 66.675)
 		(end 120.777 66.675)
@@
 	)
 	(segment
+		(start 114.5032 102.6622)
+		(end 114.5032 103.7082)
+		(width 0.25)
+		(layer "F.Cu")
+		(net 1)
+	)
+	(segment
 		(start 148.39 87.884)
 		(end 149.606 87.884)
@@
 	)
 	(via
+		(at 114.554 103.759)
+		(size 0.45)
+		(drill 0.3)
+		(layers "F.Cu" "B.Cu")
+		(net 1)
+	)
+	(via
 		(at 86.36 81.915)
 		(size 0.45)
@@
 	)
 	(segment
-		(start 124.1044 80.8247)
-		(end 128.0437 80.8247)
-		(width 0.25)
-		(layer "F.Cu")
-		(net 2)
-	)
-	(segment
 		(start 128.7138 53.0218)
 		(end 134.112 58.42)
@@
 	)
 	(segment
-		(start 123.385032 100.7872)
-		(end 114.5032 100.7872)
-		(width 0.25)
-		(layer "F.Cu")
-		(net 43)
-	)
-	(segment
-		(start 134.1345 90.037732)
-		(end 123.385032 100.7872)
-		(width 0.25)
-		(layer "F.Cu")
-		(net 43)
-	)
-	(segment
-		(start 132.317532 81.187)
-		(end 133.874468 81.187)
-		(width 0.25)
-		(layer "F.Cu")
-		(net 43)
-	)
-	(segment
-		(start 133.874468 81.187)
-		(end 134.1345 81.447032)
-		(width 0.25)
-		(layer "F.Cu")
-		(net 43)
-	)
-	(segment
-		(start 134.1345 81.447032)
-		(end 134.1345 90.037732)
-		(width 0.25)
-		(layer "F.Cu")
-		(net 43)
-	)
-	(segment
-		(start 127.40934 81.689)
-		(end 128.77966 81.689)
-		(width 0.25)
-		(layer "F.Cu")
-		(net 43)
-	)
-	(segment
-		(start 131.818132 81.6864)
-		(end 132.317532 81.187)
+		(start 146.5345 91.694)
+		(end 134.366 91.694)
 		(width 0.25)
 		(layer "F.Cu")
@@
 	)
 	(segment
-		(start 127.40674 81.6864)
-		(end 127.40934 81.689)
+		(start 134.366 91.694)
+		(end 125.2728 100.7872)
 		(width 0.25)
 		(layer "F.Cu")
@@
 	)
 	(segment
-		(start 126.8476 81.6864)
-		(end 127.40674 81.6864)
-		(width 0.25)
-		(layer "F.Cu")
-		(net 43)
-	)
-	(segment
-		(start 128.77966 81.689)
-		(end 128.78226 81.6864)
-		(width 0.25)
-		(layer "F.Cu")
-		(net 43)
-	)
-	(segment
-		(start 124.1044 82.6497)
-		(end 125.8843 82.6497)
-		(width 0.25)
-		(layer "F.Cu")
-		(net 43)
-	)
-	(segment
-		(start 125.8843 82.6497)
-		(end 126.8476 81.6864)
-		(width 0.25)
-		(layer "F.Cu")
-		(net 43)
-	)
-	(segment
-		(start 128.78226 81.6864)
-		(end 131.818132 81.6864)
+		(start 125.2728 100.7872)
+		(end 114.5032 100.7872)
 		(width 0.25)
 		(layer "F.Cu")
@@
 	)
 	(segment
-		(start 146.05 73.816)
-		(end 146.05 76.80616)
-		(width 0.25)
-		(layer "F.Cu")
-		(net 44)
-	)
-	(segment
-		(start 151.511 88.773)
-		(end 148.43724 91.84676)
-		(width 0.25)
-		(layer "F.Cu")
-		(net 44)
-	)
-	(segment
-		(start 124.21096 102.6622)
-		(end 114.5032 102.6622)
+		(start 151.892 89.281)
+		(end 151.892 81.788)
 		(width 0.25)
 		(layer "F.Cu")
@@
 	)
 	(segment
-		(start 148.43724 91.84676)
-		(end 135.0264 91.84676)
+		(start 148.3595 91.694)
+		(end 149.479 91.694)
 		(width 0.25)
 		(layer "F.Cu")
@@
 	)
 	(segment
-		(start 146.05 76.80616)
-		(end 151.511 82.26716)
+		(start 149.479 91.694)
+		(end 151.892 89.281)
 		(width 0.25)
 		(layer "F.Cu")
@@
 	)
 	(segment
-		(start 135.0264 91.84676)
-		(end 124.21096 102.6622)
+		(start 146.05 75.946)
+		(end 146.05 73.816)
 		(width 0.25)
 		(layer "F.Cu")
@@
 	)
 	(segment
-		(start 151.511 82.26716)
-		(end 151.511 88.773)
+		(start 151.892 81.788)
+		(end 146.05 75.946)
 		(width 0.25)
 		(layer "F.Cu")

Commit message: Layout improvements
Parts:
- moved R4 35.7 mm to (90.4, 69.6), turned to -90 degrees
- moved R3 33.3 mm to (90.4, 83.9)
- moved R5 0.89 mm to (112.3, 95.0), turned to -90 degrees
- moved R8 0.76 mm to (126.0, 60.7)
- moved C1 0.38 mm to (141.7, 60.8)
- moved C3 0.27 mm to (86.4, 69.6)
Routing:
- net /BMS_TX: track 92.4 -> 47.3 mm
- net VCC: track 159.1 -> 200.2 mm
- net /BMS_RX: track 82.3 -> 52.8 mm
- net Net-(U2-RA1/AN1): track 61.0 -> 84.7 mm
- net Net-(U2-RA0/AN0): track 54.3 -> 65.0 mm
- net /LCD_E: track 40.8 -> 41.9 mm
- net /BMS_FAULT: track 10.9 -> 10.0 mm
- net /LCD_RS: track 47.9 -> 48.0 mm, vias 2 -> 0
Other:
- board text added: "Tesla Model S BMB Connector Pinout"
- board text removed: "Tesla BMB Connector Pinout"

Commit message: Final fixes. Created Gerber files.
Connections:
- net Net-(DS1-LED(-)) renamed /LED-
- DS1 pad 4: /LCD_E -> /LCD_RS
- DS1 pad 6: /LCD_RS -> /LCD_E
- U2 pad 25: /LCD_E -> /LCD_RS
- U2 pad 26: /LCD_RS -> /LCD_E
Routing:
- net /LCD_RS: track 48.0 -> 41.9 mm
- net /LCD_E: track 41.9 -> 48.0 mm
Other:
- board text added: "Rev 1.0 2025"
- board text removed: "Rev 0.1 2025"
Changed lines of the file:
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@@
 	(title_block
 		(title "TeslaBMBChecker")
-		(date "2025-07-10")
-		(rev "0.1")
+		(date "2025-07-11")
+		(rev "1.0")
 	)
 	(layers
@@
 			(plot_on_all_layers_selection 0x00000000_00000000_00000000_00000000)
 			(disableapertmacros no)
-			(usegerberextensions no)
-			(usegerberattributes yes)
-			(usegerberadvancedattributes yes)
-			(creategerberjobfile yes)
+			(usegerberextensions yes)
+			(usegerberattributes no)
+			(usegerberadvancedattributes no)
+			(creategerberjobfile no)
 			(dashed_line_dash_ratio 12.000000)
 			(dashed_line_gap_ratio 3.000000)
@@
 			(sketchdnponfab yes)
 			(crossoutdnponfab yes)
-			(subtractmaskfromsilk no)
+			(subtractmaskfromsilk yes)
 			(outputformat 1)
 			(mirror no)
-			(drillshape 1)
+			(drillshape 0)
 			(scaleselection 1)
-			(outputdirectory "")
+			(outputdirectory "../Gerber/1.0/")
 		)
 	)
@@
 	(net 12 "/LCD_RS")
 	(net 13 "/LCD_E")
-	(net 14 "Net-(DS1-LED(-))")
+	(net 14 "/LED-")
 	(net 15 "/LCD_D5")
 	(net 16 "/BMS_RX")
@@
 			(layers "F.Cu" "F.Mask" "F.Paste")
 			(roundrect_rratio 0.25)
-			(net 14 "Net-(DS1-LED(-))")
+			(net 14 "/LED-")
 			(pinfunction "D")
 			(pintype "passive")
@@
 			(layers "F.Cu" "F.Mask" "F.Paste")
 			(roundrect_rratio 0.25)
-			(net 13 "/LCD_E")
+			(net 12 "/LCD_RS")
 			(pinfunction "RB4/KBI0/AN9")
 			(pintype "bidirectional")
@@
 			(layers "F.Cu" "F.Mask" "F.Paste")
 			(roundrect_rratio 0.25)
-			(net 12 "/LCD_RS")
+			(net 13 "/LCD_E")
 			(pinfunction "RB5/KBI1/PGM")
 			(pintype "bidirectional")
@@
 			(layers "*.Cu" "*.Mask" "B.SilkS")
 			(remove_unused_layers no)
-			(net 13 "/LCD_E")
+			(net 12 "/LCD_RS")
 			(pinfunction "RS")
 			(pintype "input")
@@
 			(layers "*.Cu" "*.Mask" "B.SilkS")
 			(remove_unused_layers no)
-			(net 12 "/LCD_RS")
+			(net 13 "/LCD_E")
 			(pinfunction "E")
 			(pintype "input")
@@
 			(layers "*.Cu" "*.Mask" "B.SilkS")
 			(remove_unused_layers no)
-			(net 14 "Net-(DS1-LED(-))")
+			(net 14 "/LED-")
 			(pinfunction "LED(-)")
 			(pintype "power_in")
@@
 		)
 	)
-	(gr_text "Rev 0.1   2025"
+	(gr_text "Rev 1.0   2025"
 		(at 86.868 54.61 0)
 		(layer "F.SilkS")
@@
 	)
 	(segment
-		(start 134.960968 63.19)
-		(end 133.651001 63.19)
+		(start 158.75 61.849)
+		(end 158.75 54.737)
 		(width 0.25)
 		(layer "F.Cu")
@@
 	)
 	(segment
-		(start 133.651001 63.19)
-		(end 133.35 63.491001)
+		(start 158.75 54.737)
+		(end 156.6538 52.6408)
 		(width 0.25)
 		(layer "F.Cu")
@@
 	)
 	(segment
-		(start 151.5738 50.95497)
-		(end 153.83183 53.213)
+		(start 135.763 67.945)
+		(end 152.654 67.945)
 		(width 0.25)
 		(layer "F.Cu")
@@
 	)
 	(segment
-		(start 136.226 67.519)
-		(end 135.221 66.514)
+		(start 134.62 64.516)
+		(end 134.62 66.802)
 		(width 0.25)
 		(layer "F.Cu")
@@
 	)
 	(segment
-		(start 135.221 66.514)
-		(end 135.221 63.450032)
+		(start 152.654 67.945)
+		(end 158.75 61.849)
 		(width 0.25)
 		(layer "F.Cu")
@@
 	)
 	(segment
-		(start 158.324 54.913454)
-		(end 158.324 61.672546)
+		(start 156.6538 52.6408)
+		(end 156.6538 50.20586)
 		(width 0.25)
 		(layer "F.Cu")
@@
 	)
 	(segment
-		(start 152.477546 67.519)
-		(end 136.226 67.519)
+		(start 134.62 66.802)
+		(end 135.763 67.945)
 		(width 0.25)
 		(layer "F.Cu")
@@
 	)
 	(segment
-		(start 135.221 63.450032)
-		(end 134.960968 63.19)
+		(start 134.960968 63.19)
+		(end 133.651001 63.19)
 		(width 0.25)
 		(layer "F.Cu")
-		(net 12)
+		(net 13)
 	)
 	(segment
-		(start 151.5738 50.20586)
-		(end 151.5738 50.95497)
+		(start 133.651001 63.19)
+		(end 133.35 63.491001)
 		(width 0.25)
 		(layer "F.Cu")
-		(net 12)
+		(net 13)
 	)
 	(segment
-		(start 133.35 63.491001)
-		(end 133.35 64.516)
+		(start 151.5738 50.95497)
+		(end 153.83183 53.213)
 		(width 0.25)
 		(layer "F.Cu")
-		(net 12)
+		(net 13)
 	)
 	(segment
-		(start 156.623546 53.213)
-		(end 158.324 54.913454)
+		(start 136.226 67.519)
+		(end 135.221 66.514)
 		(width 0.25)
 		(layer "F.Cu")
-		(net 12)
+		(net 13)
 	)
 	(segment
-		(start 153.83183 53.213)
-		(end 156.623546 53.213)
+		(start 135.221 66.514)
+		(end 135.221 63.450032)
 		(width 0.25)
 		(layer "F.Cu")
-		(net 12)
+		(net 13)
 	)
 	(segment
-		(start 158.324 61.672546)
-		(end 152.477546 67.519)
+		(start 158.324 54.913454)
+		(end 158.324 61.672546)
 		(width 0.25)
 		(layer "F.Cu")
-		(net 12)
+		(net 13)
 	)
 	(segment
-		(start 158.75 61.849)
-		(end 158.75 54.737)
+		(start 152.477546 67.519)
+		(end 136.226 67.519)
 		(width 0.25)
 		(layer "F.Cu")
@@
 	)
 	(segment
-		(start 158.75 54.737)
-		(end 156.6538 52.6408)
+		(start 135.221 63.450032)
+		(end 134.960968 63.19)
 		(width 0.25)
 		(layer "F.Cu")
@@
 	)
 	(segment
-		(start 135.763 67.945)
-		(end 152.654 67.945)
+		(start 151.5738 50.20586)
+		(end 151.5738 50.95497)
 		(width 0.25)
 		(layer "F.Cu")
@@
 	)
 	(segment
-		(start 134.62 64.516)
-		(end 134.62 66.802)
+		(start 133.35 63.491001)
+		(end 133.35 64.516)
 		(width 0.25)
 		(layer "F.Cu")
@@
 	)
 	(segment
-		(start 152.654 67.945)
-		(end 158.75 61.849)
+		(start 156.623546 53.213)
+		(end 158.324 54.913454)
 		(width 0.25)
 		(layer "F.Cu")
@@
 	)
 	(segment
-		(start 156.6538 52.6408)
-		(end 156.6538 50.20586)
+		(start 153.83183 53.213)
+		(end 156.623546 53.213)
 		(width 0.25)
 		(layer "F.Cu")
@@
 	)
 	(segment
-		(start 134.62 66.802)
-		(end 135.763 67.945)
+		(start 158.324 61.672546)
+		(end 152.477546 67.519)
 		(width 0.25)
 		(layer "F.Cu")
@@
 		(width 0.25)
 		(layer "F.Cu")
-		(net 18)
-	)
-	(segment
-		(start 112.268 98.171)
-		(end 112.2915 98.1475)
-		(width 0.25)
-		(layer "F.Cu")
