File: Board/TeslaBMBCheck/TeslaBMBCheck.kicad_sch (KiCad schematic)
At the start: 37 parts, among them J1 TESLA_BMS, J2 CHARGE, J9 ICSP, K2 SLA-05VDC-SL-C, Q1 IRLML2244, Q2 BSS138, Q3 IRLML2502, U1 USBLC6, U2 PIC18F2480-ISO, Y1 10 MHz

Commit message: Migrate to KiCad 10. Add 1.1 BOM
Parts:
- SW1, SW2: value ~ -> (none)
